Commit message: Update pan_tilt.urdf.xacro

File: pan_tilt_description/urdf/pan_tilt.urdf.xacro (robot description, xacro)
@@ -11,5 +11,5 @@
     <link name="${prefix}_base_link">
       <visual>
-        <origin xyz="0 0 0" rpy="0 0 ${P_PI/2}"/>
+        <origin xyz="0 0 0" rpy="0 0 -${P_PI/2}"/>
         <geometry>
           <mesh filename="package://pan_tilt_description/urdf/mesh/base.stl"/>
@@ -22,5 +22,5 @@
     <link name="${prefix}_yaw_link">
       <visual>
-        <origin xyz="0 0 0" rpy="0 0 ${P_PI/2}"/>
+        <origin xyz="0 0 0" rpy="0 0 -${P_PI/2}"/>
         <geometry>
           <mesh filename="package://pan_tilt_description/urdf/mesh/yaw.stl"/>
@@ -40,5 +40,5 @@
     <link name="${prefix}_pitch_link">
       <visual>
-        <origin xyz="0 0 0" rpy="0 0 ${P_PI/2}"/>
+        <origin xyz="0 0 0" rpy="0 0 -${P_PI/2}"/>
         <geometry>
           <mesh filename="package://pan_tilt_description/urdf/mesh/pitch.stl"/>
